File: signal_distribution_board/signal_distribution_board.kicad_pcb (KiCad board)
At the start: 2 copper layers, 107.7 x 122 mm, 18 parts, among them J1 RC1, J10 LED Power, J11 LED, J12 LED, J2 RC2, J3 RC3, J4 RC4, J5 RC5, J6 RC6, J7 Signal Input, J8 LED, J9 LED

Commit message: Updates to board routing
Parts:
- J11, J8: value LED -> LED_A
- J12, J9: value LED -> LED_B
Routing:
- net Earth: track 289.3 -> 0.00 mm
- net Net-(J11-Pin_1): track 39.7 -> 42.5 mm
- net Net-(J12-Pin_2): track 42.2 -> 44.1 mm
